Commit message: d

File: description/depth_camera.xacro (robot description, xacro)
@@ -15,5 +15,5 @@
     </link>
     <joint name="camera_optical_joint" type="fixed">
-        <parent link="camera_joint"/>
+        <parent link="camera_link"/>
         <child link="camera_link_optical"/>
         <origin xyz="0.245 0.0 0.0" rpy="${-pi/2} 0 ${-pi/2}"/>

Commit message: fix size

File: description/depth_camera.xacro (robot description, xacro)
@@ -9,5 +9,5 @@
         <visual>
             <geometry>
-                <box xyz="0.3 0.1 0.1" rpy="0 0 0"/>
+                <box size="0.3 0.1 0.1" rpy="0 0 0"/>
             </geometry>
             <material name="red"/>

Commit message: sizer

File: description/depth_camera.xacro (robot description, xacro)
@@ -9,5 +9,5 @@
         <visual>
             <geometry>
-                <box size="0.3 0.1 0.1" rpy="0 0 0"/>
+                <box size="0.1 0.1 0.1" rpy="0 0 0"/>
             </geometry>
             <material name="red"/>

Commit message: d

File: description/depth_camera.xacro (robot description, xacro)
@@ -9,5 +9,5 @@
         <visual>
             <geometry>
-                <box size="0.1 0.1 0.1" rpy="0 0 0"/>
+                <box size="0.05 0.05 0.05" rpy="0 0 0"/>
             </geometry>
             <material name="red"/>
@@ -17,5 +17,5 @@
         <parent link="camera_link"/>
         <child link="camera_link_optical"/>
-        <origin xyz="0.245 0.0 0.0" rpy="${-pi/2} 0 ${-pi/2}"/>
+        <origin xyz="0.145 0.0 0.0" rpy="${-pi/2} 0 ${-pi/2}"/>
     </joint>
     <link name="camera_link_optical"></link>

Commit message: d

File: description/depth_camera.xacro (robot description, xacro)
@@ -4,5 +4,5 @@
         <parent link="chassis"/>
         <child link="camera_link"/>
-        <origin xyz="0.245 0.0 0.0" rpy="0 0 0"/>
+        <origin xyz="0.145 0.0 0.0" rpy="0 0 0"/>
     </joint>
     <link name="camera_link">

Commit message: d

File: description/depth_camera.xacro (robot description, xacro)
@@ -4,5 +4,5 @@
         <parent link="chassis"/>
         <child link="camera_link"/>
-        <origin xyz="0.145 0.0 0.0" rpy="0 0 0"/>
+        <origin xyz="0.145 0.0 0.10" rpy="0 0 0"/>
     </joint>
     <link name="camera_link">
