Commit message: in progress of implementing the drivers in plugin

File: description/ros2_control.xacro (robot description, xacro)
@@ -1,6 +1,44 @@
 <?xml version="1.0"?>
 <robot xmlns:xacro="http://www.ros.org/wiki/xacro">
-  <ros2_control name="GazeboSystem" type="system">
+  <ros2_control name="RealRobot" type="system">
   <!-- hardware interface for the control manager-->
+    <hardware>
+      <plugin>#file location of the C++ drivers</plugin>
+    </hardware>
+    <joint name="Right_Rear_wheel_joint">
+      <command_interface name="velocity">
+        <param name="min">-10</param>
+        <param name="max">10</param>
+      </command_interface>
+      <state_interface name="velocity"/>
+      <state_interface name="position"/>
+    </joint>
+    <joint name="Right_Front_wheel_joint">
+      <command_interface name="velocity">
+        <param name="min">-10</param>
+        <param name="max">10</param>
+      </command_interface>
+      <state_interface name="velocity"/>
+      <state_interface name="position"/>
+    </joint>
+    <joint name="left_Rear_wheel_joint">
+      <command_interface name="velocity">
+        <param name="min">-10</param>
+        <param name="max">10</param>
+      </command_interface>
+      <state_interface name="velocity"/>
+      <state_interface name="position"/>
+    </joint>
+    <joint name="Left_Front_wheel_joint">
+      <command_interface name="velocity">
+        <param name="min">-10</param>
+        <param name="max">10</param>
+      </command_interface>
+      <state_interface name="velocity"/>
+      <state_interface name="position"/>
+    </joint>
+  </ros2_control>
+  <!-- <ros2_control name="GazeboSystem" type="system">
+    hardware interface for the control manager
     <hardware>
       <plugin>gazebo_ros2_control/GazeboSystem</plugin>
@@ -39,9 +77,9 @@
     </joint>
   </ros2_control>
-  <!-- Tells Gazebo to use ROS2 control-->
   <gazebo>
-    <plugin name="gazebo_ros2_control" filename="libgazebo_ros2_control.so"
+    <plugin name="gazebo_ros2_control" filename="libgazebo_ros2_control.so">
       <parameters>$(find rosx3_new)/config/my_controllers.yaml</parameters>
     </plugin>
   </gazebo>
+  -->
 </robot>
